File: power_dispatch/power_dispatch.kicad_pcb (KiCad board)
At the start: 2 copper layers, 78 x 63.5 mm, 95 parts, among them IC1 SRBH-06H1A1G, IC2 BTS500251TADATMA2, J1 Conn_01x02, J10 Conn_01x02, J11 Conn_01x02, J13 Conn_01x02, J15 USB_A, J2 Conn_01x02, J3 Conn_01x02, J4 Conn_01x02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

Commit message: Power dispatch V1.0
Parts:
- added G***: LOGO, UTCoupe:logo_UTCoupe_Big, B.Cu at (129.5, 97.6)
- added R21: NC, Resistor_SMD:R_0603_1608Metric, F.Cu at (139.7, 99.9)
- C3: value 4.7uF -> 4u7
- C8: value 150nF -> 220nF
- IC1: footprint SamacSys_Parts:SRBH06H1A1G -> UTCoupe:SRBH06H1A1G
- IC2: footprint SamacSys_Parts:IPB180N03S4L01 -> UTCoupe:IPB180N03S4L01
- J7: footprint Connector_PinHeader_2.54mm:PinHeader_1x05_P2.54mm_Vertical -> Connector_PinHeader_1.27mm:PinHeader_1x05_P1.27mm_Vertical
- R15, R16, R19: footprint Capacitor_SMD:C_0603_1608Metric -> Resistor_SMD:R_0603_1608Metric
- moved LOGO1 34.7 mm to (142.3, 71.1)
- moved G*** 1.77 mm to (134.3, 111.4)
Connections:
- D5 pad 1: CBUS0 -> CBUS1
- D6 pad 1: CBUS3 -> CBUS2
- U3 pad 15: CBUS0 -> Net-(U3-Pad15)
- U3 pad 16: CBUS3 -> Net-(U3-Pad16)
Routing:
- net CBUS2: track 0.00 -> 9.93 mm, vias 0 -> 2
- net SWO: track 22.8 -> 16.2 mm
- net SWDIO: track 18.9 -> 16.4 mm
- net CBUS3: track 2.10 -> 0.00 mm
- net CBUS1: track 0.00 -> 1.96 mm
- net CBUS0: track 1.70 -> 0.00 mm
- net +3V3: track 67.2 -> 68.6 mm
- net GND: track 222.6 -> 223.9 mm
- net NRST: track 40.4 -> 41.2 mm
Other:
- board text added: "+"
- board text added: "+5P"
- board text added: "+5V"
- board text added: "+5VL"
- board text added: "-"
- board text added: "BAT1"
- board text added: "BAT2"
- board text added: "BAU"
- board text added: "CDR2021"
- board text added: "HUB USB"
- board text added: "OUTPUT"
- board text added: "RX"
- board text added: "SWITCH"
- board text added: "TX"
- board text added: "V1.0"
- board text added: "power_dispatch"
