File: power_dispatch/power_dispatch.sch (KiCad schematic (older format))
At the start: 94 parts, among them IC1 SRBH-06H1A1G, IC2 BTS500251TADATMA2, J1 Conn_01x02, J10 Conn_01x02, J11 Conn_01x02, J13 Conn_01x02, J15 USB_A, J2 Conn_01x02, J3 Conn_01x02, J4 Conn_01x02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

Commit message: Power dispatch V1.0
Parts:
- removed IC1: SRBH-06H1A1G, SRBH06H1A1G, symbol power_dispatch-rescue:SRBH-06H1A1G-SamacSys_Parts-POWER_2-rescue-POWER_3-rescue
- removed IC2: BTS500251TADATMA2, IPB180N03S4L01, symbol power_dispatch-rescue:BTS500251TADATMA2-SamacSys_Parts-POWER_2-rescue-POWER_3-r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
- added IC1: SRBH-06H1A1G, UTCoupe:SRBH06H1A1G, symbol UTCoupe:SRBH-06H1A1G
- added IC2: BTS500251TADATMA2, UTCoupe:IPB180N03S4L01, symbol UTCoupe:BTS500251TADATMA2
- added R21: NC, Resistor_SMD:R_0603_1608Metric, symbol Device:R
- BZ1: LCSC (none) -> C94599
- C1, C13, C14, C15, C17, C18, C22, C24, C26, C4, C9: LCSC (none) -> C14663
- C10, C11: LCSC (none) -> C38523
- C12, C6: LCSC (none) -> C19666
- C16: LCSC (none) -> C15849
- C19: LCSC (none) -> C57112
- C2: LCSC (none) -> C96182
- C23, C25: LCSC (none) -> C1671
- C3: value 4.7uF -> 4u7; LCSC (none) -> C19666
- C5, C7: LCSC (none) -> C19702
- C8: value 150nF -> 220nF; LCSC (none) -> C21120
- D1, D2, D3, D4, D7, D9: LCSC (none) -> C2286
- D10: LCSC (none) -> C72043
- D5, D6: LCSC (none) -> C72041
- D8: LCSC (none) -> C81598
- F1: LCSC (none) -> C151137
- FB1: LCSC (none) -> C74480
- J6: LCSC (none) -> C91144
- J7: footprint Connector_PinHeader_2.54mm:PinHeader_1x05_P2.54mm_Vertical -> Connector_PinHeader_1.27mm:PinHeader_1x05_P1.27mm_Vertical
- L1: LCSC (none) -> C12327
- Q1: LCSC (none) -> C350312
- R1, R10, R14, R24, R26: LCSC (none) -> C22978
- R11, R13: LCSC (none) -> C21190
- R12, R2: LCSC (none) -> C23162
- R15, R16: footprint Capacitor_SMD:C_0603_1608Metric -> Resistor_SMD:R_0603_1608Metric; LCSC (none) -> C25190
- R18: LCSC (none) -> C21189
- R19: footprint Capacitor_SMD:C_0603_1608Metric -> Resistor_SMD:R_0603_1608Metric; LCSC (none) -> C23179
- R22, R23: LCSC (none) -> C22966
- R25, R27, R28, R3, R5, R6, R8: LCSC (none) -> C25804
- R4: LCSC (none) -> C4190
- R7, R9: LCSC (none) -> C22843
- SW1: LCSC (none) -> C115357
- U1, U8: LCSC (none) -> C145745
- U2: LCSC (none) -> C190642
- U5: LCSC (none) -> C5446
- Y1: LCSC (none) -> C253746
Connections:
- net +12P: now also IC2.5 (OUT_1), IC2.6 (OUT_2), IC2.7 (OUT_3)
- net +12V: now also IC1.2 (VIN)
- net +3V3: now also R21.1
- net +5VP: now also IC1.4 (VOUT)
- net +BATT: now also IC2.4 (VS)
- net CBUS1: now also D5.1 (K)
- net CBUS2: now also D6.1 (K)
- net GND: now also IC1.3 (GND), IC2.1 (GND)
- net PWRCMD: now also R21.2
- net TRIM: now also IC1.5 (TRIM)
- net at R27.2, R28.1: now also IC1.1 (REMOTE_ON/OFF)
- net at R13.2, R2.1: now also IC2.3 (IS)
- net at C8.1, R12.1: now also IC2.2 (IN)
- net CBUS0: no longer names the net of U3.15 (CBUS0)
- net CBUS0: no longer D5.1 (K)
- net CBUS3: no longer names the net of U3.16 (CBUS3)
- net CBUS3: no longer D6.1 (K)
- no-connect marks 30 -> 34
